Commit message: fix(gazebo): bolt Panda base to world and stabilize arm physics
Add world fixed joint, realistic link inertials, joint damping, and
position gain so the arm stays upright and joint trajectories execute.

Co-authored-by: Cursor <cursoragent@cursor.com>

File: ros2_ws/src/panda_sim_bringup/urdf/panda_gz.urdf.xacro (robot description, xacro)
@@ -4,4 +4,10 @@
   <xacro:property name="initial_positions" value="${xacro.load_yaml('$(find my_panda_moveit_config)/config/initial_positions.yaml')['initial_positions']}"/>
   <xacro:include filename="$(find moveit_resources_panda_description)/urdf/panda.urdf"/>
+  <!-- Fixed base: without this the whole model is a free body in Gazebo physics. -->
+  <link name="world"/>
+  <joint name="panda_world_joint" type="fixed">
+    <parent link="world"/>
+    <child link="panda_link0"/>
+  </joint>
   <ros2_control name="panda_gz_system" type="system">
     <hardware>
@@ -30,3 +36,20 @@
     </plugin>
   </gazebo>
+  <!-- Reduce joint sag before controllers claim position interfaces. -->
+  <xacro:macro name="panda_gz_joint_damping" params="joint_name">
+    <gazebo reference="${joint_name}">
+      <physics>
+        <ode>
+          <implicit_spring_damper>1</implicit_spring_damper>
+        </ode>
+      </physics>
+    </gazebo>
+  </xacro:macro>
+  <xacro:panda_gz_joint_damping joint_name="panda_joint1"/>
+  <xacro:panda_gz_joint_damping joint_name="panda_joint2"/>
+  <xacro:panda_gz_joint_damping joint_name="panda_joint3"/>
+  <xacro:panda_gz_joint_damping joint_name="panda_joint4"/>
+  <xacro:panda_gz_joint_damping joint_name="panda_joint5"/>
+  <xacro:panda_gz_joint_damping joint_name="panda_joint6"/>
+  <xacro:panda_gz_joint_damping joint_name="panda_joint7"/>
 </robot>

Commit message: fix(grasp): make inner-loop pick work end-to-end in Gazebo
Rework the simulated grasp from a broken set_pose-drag shim to Gazebo's
native DetachableJoint physical attach, and fix the upstream blockers that
kept the arm from ever reaching the block.

- urdf: declare one DetachableJoint per graspable object; parent_link must be
  panda_link7 (panda_hand/link8 collapse into it during URDF->SDF reduction).
- launch: bridge /grasp/<model>/attach|detach (Empty) and keep set_pose bridge.
- gazebo_gripper_sim: publish attach/detach instead of dragging; tighten grasp
  selection to horizontal-distance + vertical band centered on ee offset; snap
  block to gripper center before attach so it ends up gripped, not dangling;
  detach-all on open and on startup to clear stale joints across restarts.
- control: raise gz_ros2_control position gain 0.5->15 and rate 100->1000 so
  the wrist stops sagging ~3 rad under gravity (now ~0.02 rad tracking error).
- moveit_helper: vertical top-down grasp quat (was tilted 45deg, came in
  sideways); position tolerance 2cm->1cm, orientation 0.35->0.2 rad; log
  commanded-vs-reached link8 to surface constraint settling.
- executor: add target block to planning scene during approach so MoveIt routes
  around it, remove it just before the vertical descent; planning-scene attach
  is non-fatal bookkeeping.
- servo_helper: fix spin-inside-executor deadlock and undefined _check_abort
  (servo path kept as fallback; pure-MoveIt is the default).

Co-Authored-By: Claude Opus 4.8 <noreply@anthropic.com>

File: ros2_ws/src/panda_sim_bringup/urdf/panda_gz.urdf.xacro (robot description, xacro)
@@ -30,4 +30,5 @@
     <xacro:panda_gz_joint joint_name="panda_joint6"/>
     <xacro:panda_gz_joint joint_name="panda_joint7"/>
+    <xacro:panda_gz_joint joint_name="panda_finger_joint1"/>
   </ros2_control>
   <gazebo>
@@ -56,3 +57,28 @@
   <xacro:panda_gz_joint_damping joint_name="panda_joint6"/>
   <xacro:panda_gz_joint_damping joint_name="panda_joint7"/>
+  <xacro:panda_gz_joint_damping joint_name="panda_finger_joint1"/>
+  <!-- Physical grasp: one DetachableJoint per graspable object. The plugin creates a
+       real fixed joint between panda_hand and the object's link when its attach_topic
+       gets a msgs.Empty, and removes it on detach_topic. gazebo_gripper_sim.py drives
+       these topics (no more set_pose dragging). child_link is "link" for every object
+       model in pick_place_desk.sdf. -->
+  <!-- parent_link must be a link that survives URDF->SDF fixed-joint reduction in gz.
+       panda_hand / panda_link8 are fixed-jointed and get collapsed into panda_link7,
+       so the hand is rigidly part of panda_link7 — that's the valid attach parent. -->
+  <xacro:macro name="grasp_joint" params="object">
+    <gazebo>
+      <plugin filename="ignition-gazebo-detachable-joint-system"
+              name="ignition::gazebo::systems::DetachableJoint">
+        <parent_link>panda_link7</parent_link>
+        <child_model>${object}</child_model>
+        <child_link>link</child_link>
+        <attach_topic>/grasp/${object}/attach</attach_topic>
+        <detach_topic>/grasp/${object}/detach</detach_topic>
+        <output_topic>/grasp/${object}/state</output_topic>
+        <suppress_child_warning>true</suppress_child_warning>
+      </plugin>
+    </gazebo>
+  </xacro:macro>
+  <xacro:grasp_joint object="red_block_01"/>
+  <xacro:grasp_joint object="green_block_01"/>
 </robot>
