Commit message: fix(perception): calibrate Gazebo camera TF and depth back-projection
Align desk object poses with panda_link0 via range-depth unprojection, SDF
intrinsics override, and static camera TF; fix MoveIt setup assistant install,
Franka desk world merge, workspace checks, and verification scripts.

Co-authored-by: Cursor <cursoragent@cursor.com>

File: ros2_ws/src/panda_sim_bringup/urdf/overhead_camera_static.urdf (robot description, URDF)
Before this commit: robot overhead_camera_static_tf, 3 links, 2 joints
Links:
- removed link world
- added link panda_link0
Joints:
- removed joint world_to_camera_link
- added joint panda_link0_to_camera_link: type fixed, parent panda_link0, child camera_link, origin xyz=0.45 0.0 1.05 rpy=0 1.15 0

Commit message: feat(perception+mcp): real vision grounding, cross-container MCP, smoother planning
Brings the general-capability outer loop to its first real end-to-end run:
an LLM client (Claude Code over MCP) drives scan -> pick -> place on TRUE
vision instead of hardcoded coordinates, with cleaner arm trajectories.

Real perception (was: only the blue plate detected; red/green "gray"):
- The overhead camera was a 66deg oblique (pitch 1.15rad) that pushed the
  blocks off the bottom of the 480px frame — not an HSV threshold problem.
  Make it a true top-down view: pose 0.45,0,1.05/pitch1.15 -> 0.38,0,1.05/
  pitch pi/2 in pick_place_desk.sdf.
- The live camera TF comes from camera_static_tf.launch.py (NOT the urdf);
  recompute its optical-frame quaternion for straight-down viewing
  (xyzw 0.7071,-0.7071,0,0) so detections land in panda_link0 correctly.
- Depth back-projection reads the object TOP face; snap reported z to the
  object CENTER via per-label correction so grasp/place heights are right.
  Result: red/green/blue all detected, xy error <=0.6 cm, z ~0 cm.

Cross-container MCP:
- scripts/mcp_server_in_container.sh tunnels MCP stdio into the ROS
  container via `docker exec -i`, so a host MCP client (Claude Code) speaks
  to the in-container pick-place server that needs rclpy.

Smoother trajectories (was: random "abstract" joint-space detours):
- Add my_panda_moveit_config/config/ompl_planning.yaml: RRTConnect + path
  simplification + dense edge collision checking (longest_valid_segment
  0.005). This both smooths the paths and made place succeed first-try.
- Tried Pilz LIN for straight vertical moves but it was judged
  INVALID_MOTION_PLAN almost every time in a scene full of collision
  bodies; reverted to OMPL (kept the rationale in moveit_helper docstring).

Verified: S1 ("put the red block on the plate") runs end-to-end via MCP,
scan -> pick -> place, first try, all waypoints within ~1 cm.

Co-Authored-By: Claude Opus 4.8 <noreply@anthropic.com>

File: ros2_ws/src/panda_sim_bringup/urdf/overhead_camera_static.urdf (robot description, URDF)
Before this commit: robot overhead_camera_static_tf, 3 links, 2 joints
Joints:
- joint panda_link0_to_camera_link: origin xyz=0.45 0.0 1.05 rpy=0 1.15 0 -> xyz=0.38 0.0 1.05 rpy=0 1.5708 0
